Commit message: added (joined/fixed) lidar block, front arm to hold given object

File: urdf/dolly.urdf (robot description, URDF)
Before this commit: robot explorer, 4 links, 3 joints
Links:
- added link front_arm_bar, mass 1; collision box size=0.05 0.05 0.05; visual box size=0.05 0.05 0.05
- added link front_arm_bar_1, mass 1; collision box size=0.01 1 0.05; visual box size=0.01 1 0.05
- added link laser_scanner, mass 1e-5; collision box size=0.1 0.1 0.1; visual box size=0.1 0.1 0.1
Joints:
- added joint front_arm_bar_1_joint: type fixed, parent base_link, child front_arm_bar_1, origin xyz=-0.42 0.0 -0.0 rpy=0.0 0.0 0.0, axis 0.0 1 0.0
- added joint front_arm_bar_joint: type fixed, parent base_link, child front_arm_bar, origin xyz=-0.4 0.0 -0.0 rpy=0.0 0.0 0.0, axis 0.0 1 0.0
- added joint laser_scanner_joint: type fixed, parent base_link, child laser_scanner, origin xyz=-0.3 0.0 0.10 rpy=0.0 0.0 0.0, axis 0.0 1 0.0

Commit message: parent link corrected

File: urdf/dolly.urdf (robot description, URDF)
Before this commit: robot explorer, 7 links, 6 joints
Joints:
- joint front_arm_bar_1_joint: parent base_link -> base_footprint
- joint front_arm_bar_joint: parent base_link -> base_footprint
- joint laser_scanner_joint: origin xyz=-0.3 0.0 0.10 rpy=0.0 0.0 0.0 -> xyz=-0.1 0.0 0.10 rpy=0.0 0.0 0.0; parent base_link -> base_footprint

Commit message: Lidar with block has been added

File: urdf/dolly.urdf (robot description, URDF)
Before this commit: robot explorer, 7 links, 6 joints
Links:
- added link laser, mass 1; collision sphere radius=.08; visual cylinder length=0.05 radius=0.05
Joints:
- added joint laser_joint: type fixed, parent base_footprint, child laser, origin xyz=-0.1 0.0 0.16 rpy=0.0 0.0 3.14, axis 0 0 1

Commit message: Course-work world has been added to this package and re-designed the Dolly(bot) as per the world and adjusted and re-designed the front arm to hold object correctly

File: urdf/dolly.urdf (robot description, URDF)
Before this commit: robot exploDollyrer, 8 links, 7 joints
Links:
- removed link front_arm_bar_1
- added link front_arm_bar_m, mass 0.5; collision box size=0.004 0.15 0.06; visual box size=0.004 0.15 0.06
- added link front_arm_bar_r1, mass 0.5; collision box size=0.004 0.08 0.06; visual box size=0.004 0.08 0.06
- added link front_arm_bar_r2, mass 0.5; collision box size=0.004 0.08 0.06; visual box size=0.004 0.08 0.06
- added link front_arm_bar_s1, mass 0.5; collision box size=0.004 0.08 0.06; visual box size=0.004 0.08 0.06
- added link front_arm_bar_s2, mass 0.5; collision box size=0.004 0.08 0.06; visual box size=0.004 0.08 0.06
- link base_footprint: geometry collision box size=0.35 0.2 0.05; visual box size=0.35 0.2 0.05
- link caster: geometry collision sphere radius=.04; visual sphere radius=.04
- link front_arm_bar: mass 1 -> 0.5; geometry collision box size=0.025 0.025 0.025; visual box size=0.025 0.025 0.025
- link laser: mass 1 -> 0.5; geometry collision cylinder length=0.025 radius=0.025; visual cylinder length=0.025 radius=0.025
- link laser_scanner: mass 1e-5 -> 0.01; geometry collision box size=0.05 0.05 0.05; visual box size=0.05 0.05 0.05
- link wheel_left_link: mass 2 -> 1; geometry collision cylinder length=0.05 radius=0.07; visual cylinder length=0.05 radius=0.07
- link wheel_right_link: mass 2 -> 1; geometry collision cylinder length=0.05 radius=0.075; visual cylinder length=0.05 radius=0.075
Joints:
- removed joint front_arm_bar_1_joint
- added joint front_arm_bar_m_joint: type fixed, parent base_footprint, child front_arm_bar_m, origin xyz=-0.2 0.0 -0.018 rpy=0.0 0.0 0.0, axis 0.0 1 0.0
- added joint front_arm_bar_r1_joint: type fixed, parent base_footprint, child front_arm_bar_r1, origin xyz=-0.28 -0.138 -0.018 rpy=0.0 0.0 -1.578, axis 0.0 1 0.0
- added joint front_arm_bar_r2_joint: type fixed, parent base_footprint, child front_arm_bar_r2, origin xyz=-0.28 0.138 -0.018 rpy=0.0 0.0 -1.578, axis 0.0 1 0.0
- added joint front_arm_bar_s1_joint: type fixed, parent base_footprint, child front_arm_bar_s1, origin xyz=-0.22 0.105 -0.018 rpy=0.0 0.0 0.55, axis 0.0 1 0.0
- added joint front_arm_bar_s2_joint: type fixed, parent base_footprint, child front_arm_bar_s2, origin xyz=-0.22 -0.105 -0.018 rpy=0.0 0.0 -0.55, axis 0.0 1 0.0
- joint caster_joint: origin xyz=-0.3 0.0 -0.07 rpy=0.0 0.0 0.0 -> xyz=-0.135 0.0 -0.035 rpy=0.0 0.0 0.0
- joint front_arm_bar_joint: origin xyz=-0.4 0.0 -0.0 rpy=0.0 0.0 0.0 -> xyz=-0.187 0.0 -0.0 rpy=0.0 0.0 0.0
- joint laser_joint: origin xyz=-0.1 0.0 0.16 rpy=0.0 0.0 3.14 -> xyz=-0.1 0.0 0.08 rpy=0.0 0.0 3.14
- joint laser_scanner_joint: origin xyz=-0.1 0.0 0.10 rpy=0.0 0.0 0.0 -> xyz=-0.1 0.0 0.05 rpy=0.0 0.0 0.0
- joint wheel_left_joint: origin xyz=0.2 -0.25 0.0 rpy=1.57 0.0 0.0 -> xyz=0.1 -0.125 0.0 rpy=1.57 0.0 0.0
- joint wheel_right_joint: origin xyz=0.2 0.25 0.0 rpy=1.57 0.0 0.0 -> xyz=0.1 0.125 0.0 rpy=1.57 0.0 0.0

Commit message: finally assessment world is executing perfectly and Dolly is placed inside the defined world and able to move with Teleop_keyboard using 'turtlesim_teleoperation.py' by changing Ros topics from /turtle1/cmd_vel/ to /cmd_vel

File: urdf/dolly.urdf (robot description, URDF)
Before this commit: robot exploDollyrer, 12 links, 11 joints
Links:
- link laser: mass 0.5 -> 1e-5
- link laser_scanner: mass 0.01 -> 1
- link wheel_left_link: mass 1 -> 2
- link wheel_right_link: mass 1 -> 2
