Commit message: able to create a map of the world

File: urdf/dolly.urdf.xacro (robot description, xacro)
@@ -26,37 +26,37 @@
   </joint>
   <link name="base_footprint">
-    <xacro:base_inertia m="10" w="0.35" h="0.2" d="0.05"/>
+    <xacro:base_inertia m="5" w="0.35" h="0.15" d="0.03"/>
+     <visual>
+      <geometry>
+          <box size="0.35 0.2 0.03"/>
+      </geometry>
+      <material name="gray">
+        <color rgba=".2 .2 .2 1" />
+      </material>
+     </visual>
+     <collision>
+      <geometry>
+         <box size="0.35 0.2 0.03"/>
+      </geometry>
+     </collision>
+  </link>
+   <link name="wheel_right_link">
+    <xacro:cylinder_inertia m="5" r="0.0475" h="0.025"/>
     <visual>
       <geometry>
-          <box size="0.35 0.2 0.05"/>
-      </geometry>
-      <material name="gray">
-        <color rgba=".2 .2 .2 1" />
+         <cylinder radius="0.0475" length="0.025"/>
+      </geometry>
+      <material name="white">
+        <color rgba="1 1 1 1"/>
       </material>
     </visual>
     <collision>
       <geometry>
-        <box size="0.35 0.2 0.05"/>
-    </geometry>
+       <cylinder radius="0.0475" length="0.005"/>
+      </geometry>
     </collision>
-  </link>
-  <link name="wheel_right_link">
-    <xacro:cylinder_inertia m="10" r="0.0475" h="0.05"/>
-    <visual>
-      <geometry>
-          <cylinder radius="0.0475" length="0.05"/>
-      </geometry>
-      <material name="white">
-        <color rgba="1 1 1 1"/>
-      </material>
-    </visual>
-    <collision>
-      <geometry>
-        <cylinder radius="0.0475" length="0.05"/>
-      </geometry>
-    </collision>
-  </link>
+   </link>
   <joint name="wheel_right_joint" type="continuous">
-    <origin xyz="0.1 0.125 -0.015" rpy="1.57 0.0 0.0"/>
+    <origin xyz="0.1 0.115 -0.015" rpy="1.57 0.0 0.0"/>
     <parent link="base_footprint"/>
     <child link="wheel_right_link"/>
@@ -64,8 +64,8 @@
   </joint>
   <link name="wheel_left_link">
-    <xacro:cylinder_inertia m="10" r="0.0475" h="0.05"/>
+    <xacro:cylinder_inertia m="5" r="0.0475" h="0.025"/>
     <visual>
       <geometry>
-          <cylinder radius="0.0475" length="0.05"/>
+          <cylinder radius="0.0475" length="0.025"/>
       </geometry>
       <material name="white">
@@ -75,10 +75,10 @@
     <collision>
       <geometry>
-        <cylinder radius="0.0475" length="0.05"/>
+        <cylinder radius="0.0475" length="0.025"/>
       </geometry>
     </collision>
   </link>
   <joint name="wheel_left_joint" type="continuous">
-    <origin xyz="0.1 -0.125 -0.015" rpy="1.57 0.0 0.0"/>
+    <origin xyz="0.1 -0.115 -0.015" rpy="1.57 0.0 0.0"/>
     <parent link="base_footprint"/>
     <child link="wheel_left_link"/>
@@ -105,217 +105,202 @@
     <child link="caster"/>
   </joint>
-  <!--Front arm-->
-  <link name="front_arm_bar">
-    <visual>
-        <geometry>
-            <box size="0.025 0.025 0.025"/>
-        </geometry>
-        <material name="gray">
-          <color rgba=".2 .2 .2 1" />
-        </material>
-    </visual>
-    <collision>
-      <geometry>
-        <box size="0.025 0.025 0.025"/>
-      </geometry>
-    </collision>
-    <inertial>
-        <mass value="0.5"/>
-        <inertia ixx="0.01" ixy="0.0" ixz="0" iyy="0.01" iyz="0" izz="0.01" />
-    </inertial>
-  </link>
-  <joint name="front_arm_bar_joint" type="fixed">
-    <axis xyz="0.0 1 0.0"/>
-    <parent link="base_footprint"/>
-    <child link="front_arm_bar"/>
-    <origin xyz="-0.187 0.0 -0.0" rpy="0.0 0.0 0.0"/>
-  </joint>
-  <!--==========================================================-->
-  <link name="front_arm_bar_m">
-    <visual>
-        <geometry>
-            <box size="0.004 0.1 0.06"/>
-        </geometry>
-        <material name="gray">
-          <color rgba=".2 .2 .2 1" />
-        </material>
-    </visual>
-    <collision>
-      <geometry>
-        <box size="0.004 0.15 0.06"/>
-      </geometry>
-    </collision>
-    <inertial>
-      <mass value="0.5"/>
-      <inertia ixx="0.01" ixy="0.0" ixz="0" iyy="0.01" iyz="0" izz="0.01" />
-    </inertial>
-  </link>
-  <joint name="front_arm_bar_m_joint" type="fixed">
-    <axis xyz="0.0 1 0.0"/>
-    <parent link="base_footprint"/>
-    <child link="front_arm_bar_m"/>
-    <origin xyz="-0.2 0.0 -0.018" rpy="0.0 0.0 0.0"/>
-  </joint>
-  <!--==========================================================-->
-  <link name="front_arm_bar_s1">
-    <visual>
-        <geometry>
-            <box size="0.004 0.08 0.06"/>
-        </geometry>
-        <material name="gray">
-          <color rgba=".2 .2 .2 1" />
-        </material>
-    </visual>
-    <collision>
-      <geometry>
-        <box size="0.004 0.08 0.06"/>
-      </geometry>
-    </collision>
-    <inertial>
-      <mass value="0.5"/>
-      <inertia ixx="0.01" ixy="0.0" ixz="0" iyy="0.01" iyz="0" izz="0.01" />
-    </inertial>
-  </link>
-  <joint name="front_arm_bar_s1_joint" type="fixed">
-    <axis xyz="0.0 1 0.0"/>
-    <parent link="base_footprint"/>
-    <child link="front_arm_bar_s1"/>
-    <origin xyz="-0.22 0.082 -0.018" rpy="0.0 0.0 0.55"/>
-  </joint>
-  <!--==========================================================-->
-  <link name="front_arm_bar_s2">
-    <visual>
-        <geometry>
-            <box size="0.004 0.08 0.06"/>
-        </geometry>
-        <material name="gray">
-          <color rgba=".2 .2 .2 1" />
-        </material>
-    </visual>
-    <collision>
-      <geometry>
-        <box size="0.004 0.08 0.06"/>
-      </geometry>
-    </collision>
-    <inertial>
-      <mass value="0.5"/>
-      <inertia ixx="0.01" ixy="0.0" ixz="0" iyy="0.01" iyz="0" izz="0.01" />
-    </inertial>
-  </link>
-  <joint name="front_arm_bar_s2_joint" type="fixed">
-    <axis xyz="0.0 1 0.0"/>
-    <parent link="base_footprint"/>
-    <child link="front_arm_bar_s2"/>
-    <origin xyz="-0.22 -0.082 -0.018" rpy="0.0 0.0 -0.55"/>
-  </joint>
-  <!--==========================================================-->
-  <link name="front_arm_bar_r1">
-    <visual>
-        <geometry>
-            <box size="0.004 0.05 0.06"/>
-        </geometry>
-        <material name="gray">
-          <color rgba=".2 .2 .2 1" />
-        </material>
-    </visual>
-    <collision>
-      <geometry>
-        <box size="0.004 0.05 0.06"/>
-      </geometry>
-    </collision>
-    <inertial>
-      <mass value="0.5"/>
-      <inertia ixx="0.01" ixy="0.0" ixz="0" iyy="0.01" iyz="0" izz="0.01" />
-    </inertial>
-  </link>
-  <joint name="front_arm_bar_r1_joint" type="fixed">
-    <axis xyz="0.0 1 0.0"/>
-    <parent link="base_footprint"/>
-    <child link="front_arm_bar_r1"/>
-    <origin xyz="-0.265 -0.115 -0.018" rpy="0.0 0.0 -1.578"/>
-  </joint>
-  <!--==========================================================-->
-  <link name="front_arm_bar_r2">
-    <visual>
-        <geometry>
-            <box size="0.004 0.05 0.06"/>
-        </geometry>
-        <material name="gray">
-          <color rgba=".2 .2 .2 1" />
-        </material>
-    </visual>
-    <collision>
-      <geometry>
-        <box size="0.004 0.05 0.06"/>
-      </geometry>
-    </collision>
-    <inertial>
-      <mass value="0.5"/>
-      <inertia ixx="0.01" ixy="0.0" ixz="0" iyy="0.01" iyz="0" izz="0.01" />
-    </inertial>
-  </link>
-  <joint name="front_arm_bar_r2_joint" type="fixed">
-    <axis xyz="0.0 1 0.0"/>
-    <parent link="base_footprint"/>
-    <child link="front_arm_bar_r2"/>
-    <origin xyz="-0.265 0.115 -0.018" rpy="0.0 0.0 -1.578"/>
-  </joint>
-  <!--==========================================================-->
-  <!-- laser -->
-  <link name="laser">
-    <inertial>
-      <mass value="1e-5"/>
-      <inertia ixx="1e-6" ixy="0" ixz="0.0" iyy="1e-6" iyz="0.0" izz="1e-6"/>
-    </inertial>
-    <visual>
-      <geometry>
-        <cylinder radius="0.025" length="0.025"/>
-       </geometry>
-    </visual>
-    <collision>
-      <origin/>
-      <geometry>
-        <cylinder radius="0.025" length="0.025"/>
-      </geometry>
-    </collision>
-  </link>
-  <joint name="laser_joint" type="fixed">
-    <origin xyz="-0.1 0.0 0.038" rpy="0.0 0.0 3.14"/>
-    <axis xyz="0 0 1" />
-    <parent link="base_footprint"/>
-    <child link="laser"/>
-  </joint>
-  <gazebo reference="laser">
-    <sensor type="ray" name="laser">
-        <pose>0 0 0 0 0 0</pose>
-        <visualize>true</visualize>
-        <update_rate>40</update_rate>
-        <ray>
-            <scan>
-                <horizontal>
-                    <samples>720</samples>
-                    <resolution>0.1</resolution>
-                    <min_angle>-1.578</min_angle>
-                    <max_angle>1.578</max_angle>
-                </horizontal>
-            </scan>
-            <range>
-                <min>0.1</min>
-                <max>2</max>
-                <resolution>0.1</resolution>
-            </range>
-        </ray>
-        <plugin name="laser_controller" filename="libgazebo_ros_laser.so">
-            <topicName>/scan</topicName>
-            <frameName>laser</frameName>
-        </plugin>
-    </sensor>
-  </gazebo>
-  <!-- DIFFENERNTIAL DRIVEEEEEEEEEEEEE -->
-  <gazebo>
+<!--Front arm-->
+<link name="front_arm_bar">
+  <visual>
+      <geometry>
+          <box size="0.025 0.025 0.025"/>
+      </geometry>
+      <material name="gray">
+        <color rgba=".2 .2 .2 1" />
+      </material>
+  </visual>
+  <collision>
+    <geometry>
+      <box size="0.025 0.025 0.025"/>
+    </geometry>
+  </collision>
+  <xacro:base_inertia m="1" w="0.025" h="0.025" d="0.025"/>
+</link>
+<joint name="front_arm_bar_joint" type="fixed">
+  <axis xyz="0.0 1 0.0"/>
+  <parent link="base_footprint"/>
+  <child link="front_arm_bar"/>
+  <origin xyz="-0.187 0.0 -0.0" rpy="0.0 0.0 0.0"/>
+</joint>
+<!--==========================================================-->
+<link name="front_arm_bar_m">
+  <visual>
+      <geometry>
+          <box size="0.004 0.15 0.06"/>
+      </geometry>
+      <material name="gray">
+        <color rgba=".2 .2 .2 1" />
+      </material>
+  </visual>
+  <collision>
+    <geometry>
+      <box size="0.004 0.15 0.06"/>
+    </geometry>
+  </collision>
+  <xacro:base_inertia m="0.5" w="0.004" h="0.15" d="0.06"/>
+</link>
+<joint name="front_arm_bar_m_joint" type="fixed">
+  <axis xyz="0.0 1 0.0"/>
+  <parent link="base_footprint"/>
+  <child link="front_arm_bar_m"/>
+  <origin xyz="-0.2 0.0 -0.018" rpy="0.0 0.0 0.0"/>
+</joint>
+<!--==========================================================-->
+<link name="front_arm_bar_s1">
+  <visual>
+      <geometry>
+          <box size="0.004 0.08 0.06"/>
+      </geometry>
+      <material name="gray">
+        <color rgba=".2 .2 .2 1" />
+      </material>
+  </visual>
+  <collision>
+    <geometry>
+      <box size="0.004 0.08 0.06"/>
+    </geometry>
+  </collision>
+  <xacro:base_inertia m="0.5" w="0.004" h="0.08" d="0.06"/>
+</link>
+<joint name="front_arm_bar_s1_joint" type="fixed">
+  <axis xyz="0.0 1 0.0"/>
+  <parent link="base_footprint"/>
+  <child link="front_arm_bar_s1"/>
+  <origin xyz="-0.22 0.105 -0.018" rpy="0.0 0.0 0.55"/>
+</joint>
+<!--==========================================================-->
+<link name="front_arm_bar_s2">
+  <visual>
+      <geometry>
+          <box size="0.004 0.08 0.06"/>
+      </geometry>
+      <material name="gray">
+        <color rgba=".2 .2 .2 1" />
+      </material>
+  </visual>
+  <collision>
+    <geometry>
+      <box size="0.004 0.08 0.06"/>
+    </geometry>
+  </collision>
+  <xacro:base_inertia m="0.5" w="0.004" h="0.08" d="0.06"/>
+</link>
+<joint name="front_arm_bar_s2_joint" type="fixed">
+  <axis xyz="0.0 1 0.0"/>
+  <parent link="base_footprint"/>
+  <child link="front_arm_bar_s2"/>
+  <origin xyz="-0.22 -0.105 -0.018" rpy="0.0 0.0 -0.55"/>
+</joint>
+<!--==========================================================-->
+<link name="front_arm_bar_r1">
+  <visual>
+      <geometry>
+          <box size="0.004 0.08 0.06"/>
+      </geometry>
+      <material name="gray">
+        <color rgba=".2 .2 .2 1" />
+      </material>
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
Commit message: modifying the bot

File: urdf/dolly.urdf.xacro (robot description, xacro)
@@ -41,5 +41,5 @@
      </collision>
   </link>
-   <link name="wheel_right_link">
+  <link name="wheel_right_link">
     <xacro:cylinder_inertia m="5" r="0.0475" h="0.025"/>
     <visual>
@@ -56,5 +56,5 @@
       </geometry>
     </collision>
-   </link>
+  </link>
   <joint name="wheel_right_joint" type="continuous">
     <origin xyz="0.1 0.115 -0.015" rpy="1.57 0.0 0.0"/>
@@ -85,4 +85,47 @@
     <axis xyz="0.0 0.0 1.0"/>
   </joint>
+  <!-- This block connects the wheel joint to an actuator (motor), which informs both
+simulation and visualization of the robot -->
+<!--########################## BASE TRANSMISSIONS ############################################-->
+<transmission name="front_left_wheel_trans" type="SimpleTransmission">
+  <type>transmission_interface/SimpleTransmission</type>
+  <actuator name="front_left_wheel_motor">
+   <hardwareInterface>hardware_interface/VelocityJointInterface</hardwareInterface>
+   <mechanicalReduction>1</mechanicalReduction>
+  </actuator>
+  <joint name="front_left_wheel_joint">
+   <hardwareInterface>hardware_interface/VelocityJointInterface</hardwareInterface>
+  </joint>
+</transmission>
+<transmission name="front_right_wheel_trans" type="SimpleTransmission">
+  <type>transmission_interface/SimpleTransmission</type>
+  <actuator name="front_right_wheel_motor">
+   <hardwareInterface>hardware_interface/VelocityJointInterface</hardwareInterface>
+   <mechanicalReduction>1</mechanicalReduction>
+  </actuator>
+  <joint name="front_right_wheel_joint">
+   <hardwareInterface>hardware_interface/VelocityJointInterface</hardwareInterface>
+  </joint>
+</transmission>
+<transmission name="rear_left_wheel_trans" type="SimpleTransmission">
+  <type>transmission_interface/SimpleTransmission</type>
+  <actuator name="rear_left_wheel_motor">
+   <hardwareInterface>hardware_interface/VelocityJointInterface</hardwareInterface>
+   <mechanicalReduction>1</mechanicalReduction>
+  </actuator>
+  <joint name="rear_left_wheel_joint">
+   <hardwareInterface>hardware_interface/VelocityJointInterface</hardwareInterface>
+  </joint>
+</transmission>
+<transmission name="rear_right_wheel_trans" type="SimpleTransmission">
+  <type>transmission_interface/SimpleTransmission</type>
+  <actuator name="rear_right_wheel_motor">
+   <hardwareInterface>hardware_interface/VelocityJointInterface</hardwareInterface>
+   <mechanicalReduction>1</mechanicalReduction>
+  </actuator>
+  <joint name="rear_right_wheel_joint">
+   <hardwareInterface>hardware_interface/VelocityJointInterface</hardwareInterface>
+  </joint>
+</transmission>
   <link name="caster">
     <xacro:sphere_inertia m="5" r="0.03"/>
@@ -146,5 +189,5 @@
 </link>
 <joint name="front_arm_bar_m_joint" type="fixed">
-  <axis xyz="0.0 1 0.0"/>
+  <axis xyz="0.0 0 0.0"/>
   <parent link="base_footprint"/>
   <child link="front_arm_bar_m"/>
@@ -169,8 +212,8 @@
 </link>
 <joint name="front_arm_bar_s1_joint" type="fixed">
-  <axis xyz="0.0 1 0.0"/>
+  <axis xyz="0.0 0 0.0"/>
   <parent link="base_footprint"/>
   <child link="front_arm_bar_s1"/>
-  <origin xyz="-0.22 0.105 -0.018" rpy="0.0 0.0 0.55"/>
+  <origin xyz="-0.18 0.105 -0.018" rpy="0 0 -0.55"/>
 </joint>
 <!--==========================================================-->
@@ -192,8 +235,8 @@
 </link>
 <joint name="front_arm_bar_s2_joint" type="fixed">
-  <axis xyz="0.0 1 0.0"/>
+  <axis xyz="0.0 0 0.0"/>
   <parent link="base_footprint"/>
   <child link="front_arm_bar_s2"/>
-  <origin xyz="-0.22 -0.105 -0.018" rpy="0.0 0.0 -0.55"/>
+  <origin xyz="-0.18 -0.105 -0.018" rpy="0.0 0.0 0.55"/>
 </joint>
 <!--==========================================================-->
@@ -215,8 +258,8 @@
 </link>
 <joint name="front_arm_bar_r1_joint" type="fixed">
-  <axis xyz="0.0 1 0.0"/>
+  <axis xyz="0.0 0 0.0"/>
   <parent link="base_footprint"/>
   <child link="front_arm_bar_r1"/>
-  <origin xyz="-0.28 -0.138 -0.018" rpy="0.0 0.0 -1.578"/>
+  <origin xyz="-0.12 -0.138 -0.018" rpy="0.0 0.0 -1.578"/>
 </joint>
 <!--==========================================================-->
@@ -238,8 +281,8 @@
 </link>
 <joint name="front_arm_bar_r2_joint" type="fixed">
-  <axis xyz="0.0 1 0.0"/>
+  <axis xyz="0.0 0 0.0"/>
   <parent link="base_footprint"/>
   <child link="front_arm_bar_r2"/>
-  <origin xyz="-0.28 0.138 -0.018" rpy="0.0 0.0 -1.578"/>
+  <origin xyz="-0.12 0.138 -0.018" rpy="0.0 0.0 -1.578"/>
 </joint>
 <!--==========================================================-->
@@ -305,5 +348,5 @@
       <leftJoint>wheel_left_joint</leftJoint>
       <rightJoint>wheel_right_joint</rightJoint>
-      <wheelSeparation>0.125</wheelSeparation>
+      <wheelSeparation>0.34</wheelSeparation>
       <wheelDiameter>0.095</wheelDiameter>
       <torque>20</torque>
@@ -312,4 +355,5 @@
       <publishWheelJointState>true</publishWheelJointState>
       <wheelAcceleration>2</wheelAcceleration>
+      <publishWheelTF>false</publishWheelTF>
   </plugin>
 </gazebo>
@@ -322,7 +366,17 @@
   </gazebo>
   <gazebo reference="wheel_right_link">
+    <mu1 value="1.0"/>
+    <mu2 value="1.0"/>
+    <kp value="10000000.0" />
+    <kd value="1.0" />
+    <fdir1 value="1 0 0"/>
     <material>Gazebo/Blue</material>
   </gazebo>
   <gazebo reference="wheel_left_link">
+    <mu1 value="1.0"/>
+    <mu2 value="1.0"/>
+    <kp value="10000000.0" />
+    <kd value="1.0" />
+    <fdir1 value="1 0 0"/>
     <material>Gazebo/Blue</material>
   </gazebo>
@@ -330,3 +384,11 @@
     <material>Gazebo/Red</material>
   </gazebo>
+  <!--######################################################################-->
+<gazebo>
+  <plugin name="gazebo_ros_control" filename="libgazebo_ros_control.so">
+    <robotNamespace>/</robotNamespace>
+    <controlPeriod>0.001</controlPeriod>
+    <legacyModeNS>false</legacyModeNS>
+  </plugin>
+</gazebo>
 </robot>

Commit message: added 4 wheel

File: urdf/dolly.urdf.xacro (robot description, xacro)
@@ -41,5 +41,5 @@
      </collision>
   </link>
-  <link name="wheel_right_link">
+  <link name="front_left_wheel_link">
     <xacro:cylinder_inertia m="5" r="0.0475" h="0.025"/>
     <visual>
@@ -57,11 +57,11 @@
     </collision>
   </link>
-  <joint name="wheel_right_joint" type="continuous">
+  <joint name="front_left_wheel_joint" type="continuous">
     <origin xyz="0.1 0.115 -0.015" rpy="1.57 0.0 0.0"/>
     <parent link="base_footprint"/>
-    <child link="wheel_right_link"/>
+    <child link="front_left_wheel_link"/>
     <axis xyz="0.0 0.0 1.0"/>
   </joint>
-  <link name="wheel_left_link">
+  <link name="front_right_wheel_link">
     <xacro:cylinder_inertia m="5" r="0.0475" h="0.025"/>
     <visual>
@@ -79,8 +79,52 @@
     </collision>
   </link>
-  <joint name="wheel_left_joint" type="continuous">
+  <joint name="front_right_wheel_joint" type="continuous">
     <origin xyz="0.1 -0.115 -0.015" rpy="1.57 0.0 0.0"/>
     <parent link="base_footprint"/>
-    <child link="wheel_left_link"/>
+    <child link="front_right_wheel_link"/>
+    <axis xyz="0.0 0.0 1.0"/>
+  </joint>
+  <link name="rear_left_wheel_link">
+    <xacro:cylinder_inertia m="5" r="0.0475" h="0.025"/>
+    <visual>
+      <geometry>
+         <cylinder radius="0.0475" length="0.025"/>
+      </geometry>
+      <material name="white">
+        <color rgba="1 1 1 1"/>
+      </material>
+    </visual>
+    <collision>
+      <geometry>
+       <cylinder radius="0.0475" length="0.005"/>
+      </geometry>
+    </collision>
+  </link>
+  <joint name="rear_left_wheel_joint" type="continuous">
+    <origin xyz="-0.1 0.115 -0.015" rpy="1.57 0.0 0.0"/>
+    <parent link="base_footprint"/>
+    <child link="rear_left_wheel_link"/>
+    <axis xyz="0.0 0.0 1.0"/>
+  </joint>
+  <link name="rear_right_wheel_link">
+    <xacro:cylinder_inertia m="5" r="0.0475" h="0.025"/>
+    <visual>
+      <geometry>
+          <cylinder radius="0.0475" length="0.025"/>
+      </geometry>
+      <material name="white">
+        <color rgba="1 1 1 1"/>
+      </material>
+    </visual>
+    <collision>
+      <geometry>
+        <cylinder radius="0.0475" length="0.025"/>
+      </geometry>
+    </collision>
+  </link>
+  <joint name="rear_right_wheel_joint" type="continuous">
+    <origin xyz="-0.1 -0.115 -0.015" rpy="1.57 0.0 0.0"/>
+    <parent link="base_footprint"/>
+    <child link="rear_right_wheel_link"/>
     <axis xyz="0.0 0.0 1.0"/>
   </joint>
@@ -128,24 +172,4 @@
   </joint>
 </transmission>
-  <link name="caster">
-    <xacro:sphere_inertia m="5" r="0.03"/>
-    <visual>
-      <geometry>
-        <sphere radius="0.03" />
-      </geometry>
-      <material name="white" />
-    </visual>
-    <collision>
-      <geometry>
-        <sphere radius="0.03" />
-      </geometry>
-    </collision>
-  </link>
-  <joint name="caster_joint" type="continuous">
-    <origin xyz="-0.135 0.0 -0.035" rpy="0.0 0.0 0.0"/>
-    <axis xyz="0 0 1" />
-    <parent link="base_footprint"/>
-    <child link="caster"/>
-  </joint>
 <!--Front arm-->
 <link name="front_arm_bar">
