Commit message: added new arm to hold the object

File: urdf/dolly.urdf.xacro (robot description, xacro)
@@ -56,177 +56,33 @@
     </collision>
 </link>
-<link name="front_left_wheel">
-    <inertial>
-      <origin
-        xyz="-4.1867E-18 0.0068085 -1.65658661799998E-18"
-        rpy="0 0 0" />
-      <mass
-        value="2.6578" />
-      <inertia
-        ixx="0.00856502765719703"
-        ixy="1.5074118157338E-19"
-        ixz="-4.78150098725052E-19"
-        iyy="0.013670640432096"
-        iyz="-2.68136447099727E-19"
-        izz="0.00856502765719703" />
-    </inertial>
-    <visual>
-      <origin
-        xyz="0 0 0"
-        rpy="1.5707963267949 0 0" />
-      <geometry>
-        <mesh filename="package://explorer_bot/models/world/meshes/wheel.stl" scale="0.8 0.8 0.8"/>
-      </geometry>
-      <material
-        name="">
-        <color
-          rgba="0.79216 0.81961 0.93333 1" />
-      </material>
-    </visual>
-    <collision>
-      <origin
-        xyz="0 0 0"
-        rpy="1.5707963267949 0 0" />
-      <geometry>
-        <mesh filename="package://explorer_bot/models/world/meshes/wheel.stl" scale="0.8 0.8 0.8"/>
-      </geometry>
-    </collision>
-  </link>
-<link name="front_right_wheel">
-    <inertial>
-      <origin
-        xyz="-4.1867E-18 0.0068085 -1.65658661799998E-18"
-        rpy="0 0 0" />
-      <mass
-        value="2.6578" />
-      <inertia
-        ixx="0.00856502765719703"
-        ixy="1.5074118157338E-19"
-        ixz="-4.78150098725052E-19"
-        iyy="0.013670640432096"
-        iyz="-2.68136447099727E-19"
-        izz="0.00856502765719703" />
-    </inertial>
-    <visual>
-      <origin
-        xyz="0 0 0"
-        rpy="1.5707963267949 0 0" />
-      <geometry>
-        <mesh filename="package://explorer_bot/models/world/meshes/wheel.stl" scale="0.8 0.8 0.8"/>
-      </geometry>
-      <material
-        name="">
-        <color
-          rgba="0.79216 0.81961 0.93333 1" />
-      </material>
-    </visual>
-    <collision>
-      <origin
-        xyz="0 0 0"
-        rpy="1.5707963267949 0 0" />
-      <geometry>
-        <mesh filename="package://explorer_bot/models/world/meshes/wheel.stl" scale="0.8 0.8 0.8"/>
-      </geometry>
-    </collision>
-  </link>
-<link name="rear_left_wheel">
-    <inertial>
-      <origin
-        xyz="-4.1867E-18 0.0068085 -1.65658661799998E-18"
-        rpy="0 0 0" />
-      <mass
-        value="2.6578" />
-      <inertia
-        ixx="0.00856502765719703"
-        ixy="1.5074118157338E-19"
-        ixz="-4.78150098725052E-19"
-        iyy="0.013670640432096"
-        iyz="-2.68136447099727E-19"
-        izz="0.00856502765719703" />
-    </inertial>
-    <visual>
-      <origin
-        xyz="0 0 0"
-        rpy="1.5707963267949 0 0" />
-      <geometry>
-        <mesh filename="package://explorer_bot/models/world/meshes/wheel.stl" scale="0.8 0.8 0.8"/>
-      </geometry>
-      <material
-        name="">
-        <color
-          rgba="0.79216 0.81961 0.93333 1" />
-      </material>
-    </visual>
-    <collision>
-      <origin
-        xyz="0 0 0"
-        rpy="1.5707963267949 0 0" />
-      <geometry>
-        <mesh filename="package://explorer_bot/models/world/meshes/wheel.stl" scale="0.8 0.8 0.8"/>
-      </geometry>
-    </collision>
-  </link>
-<link name="rear_right_wheel">
-    <inertial>
-      <origin
-        xyz="-4.1867E-18 0.0068085 -1.65658661799998E-18"
-        rpy="0 0 0" />
-      <mass
-        value="2.6578" />
-      <inertia
-        ixx="0.00856502765719703"
-        ixy="1.5074118157338E-19"
-        ixz="-4.78150098725052E-19"
-        iyy="0.013670640432096"
-        iyz="-2.68136447099727E-19"
-        izz="0.00856502765719703" />
-    </inertial>
-    <visual>
-      <origin
-        xyz="0 0 0"
-        rpy="1.5707963267949 0 0" />
-      <geometry>
-        <mesh filename="package://explorer_bot/models/world/meshes/wheel.stl" scale="0.8 0.8 0.8"/>
-      </geometry>
-      <material
-        name="">
-        <color
-          rgba="0.79216 0.81961 0.93333 1" />
-      </material>
-    </visual>
-    <collision>
-      <origin
-        xyz="0 0 0"
-        rpy="1.5707963267949 0 0" />
-      <geometry>
-        <mesh filename="package://explorer_bot/models/world/meshes/wheel.stl" scale="0.8 0.8 0.8"/>
-      </geometry>
-    </collision>
-  </link>
-<joint name="front_left_wheel_joint" type="continuous">
-    <axis xyz="0 1 0"/>
-    <parent link ="base_link"/>
-    <child link ="front_left_wheel"/>
-    <origin rpy ="0 0 0" xyz= "0.176 0.205 0"/>
-  </joint>
-<joint name="front_right_wheel_joint" type="continuous">
-    <axis xyz="0 1 0"/>
-    <parent link ="base_link"/>
-    <child link ="front_right_wheel"/>
-    <origin rpy ="0 0 0" xyz= "0.176 -0.205 0"/>
-  </joint>
-<joint name="rear_left_wheel_joint" type="continuous">
-    <axis xyz="0 1 0"/>
-    <parent link ="base_link"/>
-    <child link ="rear_left_wheel"/>
-    <origin rpy ="0 0 0" xyz= "-0.176 0.205 0"/>
-  </joint>
-<joint name="rear_right_wheel_joint" type="continuous">
-    <axis xyz="0 1 0"/>
-    <parent link ="base_link"/>
-    <child link ="rear_right_wheel"/>
-    <origin rpy ="0 0 0" xyz= "-0.176 -0.205 0"/>
-</joint>
-<link name="arm_base">
+<link name="arm_link">
+  <visual>
+    <origin rpy="0 0 0" xyz="0 0 0.1585"/>
+    <geometry>
+      <box size="0.0356 0.05 0.3"/>
+    </geometry>
+  </visual>
+  <collision>
+    <origin rpy="0 0 0" xyz="0 0 0.1585"/>
+    <geometry>
+      <box size="0.0356 0.05 0.3"/>
+    </geometry>
+  </collision>
+  <inertial>
+    <!-- CENTER OF MASS -->
+    <mass value="0.29302326"/>
+    <!-- box inertia: 1/12*m(y^2+z^2), ... -->
+    <inertia ixx="0.00251484771035" ixy="0" ixz="0" iyy="0.00248474836108" iyz="0" izz="9.19936757328e-05"/>
+  </inertial>
+</link>
+<joint name="arm_joint" type="continuous">
+  <parent link="base_link"/>
+  <child link="arm_link"/>
+  <dynamics damping="3.0" friction="0.3"/>
+  <limit effort="30.0" lower="-1.57079632679" upper="1.57079632679" velocity="5.0"/>
+  <origin rpy="0 0 0" xyz="-0.05 0 0.1"/>
+  <axis xyz="0 1 0"/>
+</joint>
+<link name="hand">
   <inertial>
     <origin
@@ -265,9 +121,181 @@
   </collision>
 </link>
-<joint name="arm_base_joint" type="continuous">
+<joint name="hand_joint" type="fixed">
   <axis xyz="0 0 1"/>
   <parent link="base_link"/>
-  <child link="arm_base"/>
-  <origin rpy="3.14 0 0" xyz="-0.1 0.2 0.2"/>
+  <child link="hand"/>
+  <origin rpy="0 1.578 3.14" xyz="0.05 0.27 0.2"/>
+</joint>
+<link name="front_left_wheel">
+    <inertial>
+      <origin
+        xyz="-4.1867E-18 0.0068085 -1.65658661799998E-18"
+        rpy="0 0 0" />
+      <mass
+        value="2.6578" />
+      <inertia
+        ixx="0.00856502765719703"
+        ixy="1.5074118157338E-19"
+        ixz="-4.78150098725052E-19"
+        iyy="0.013670640432096"
+        iyz="-2.68136447099727E-19"
+        izz="0.00856502765719703" />
+    </inertial>
+    <visual>
+      <origin
+        xyz="0 0 0"
+        rpy="1.5707963267949 0 0" />
+      <geometry>
+        <mesh filename="package://explorer_bot/models/world/meshes/wheel.stl" scale="0.8 0.8 0.8"/>
+      </geometry>
+      <material
+        name="">
+        <color
+          rgba="0.79216 0.81961 0.93333 1" />
+      </material>
+    </visual>
+    <collision>
+      <origin
+        xyz="0 0 0"
+        rpy="1.5707963267949 0 0" />
+      <geometry>
+        <mesh filename="package://explorer_bot/models/world/meshes/wheel.stl" scale="0.8 0.8 0.8"/>
+      </geometry>
+    </collision>
+  </link>
+<link name="front_right_wheel">
+    <inertial>
+      <origin
+        xyz="-4.1867E-18 0.0068085 -1.65658661799998E-18"
+        rpy="0 0 0" />
+      <mass
+        value="2.6578" />
+      <inertia
+        ixx="0.00856502765719703"
+        ixy="1.5074118157338E-19"
+        ixz="-4.78150098725052E-19"
+        iyy="0.013670640432096"
+        iyz="-2.68136447099727E-19"
+        izz="0.00856502765719703" />
+    </inertial>
+    <visual>
+      <origin
+        xyz="0 0 0"
+        rpy="1.5707963267949 0 0" />
+      <geometry>
+        <mesh filename="package://explorer_bot/models/world/meshes/wheel.stl" scale="0.8 0.8 0.8"/>
+      </geometry>
+      <material
+        name="">
+        <color
+          rgba="0.79216 0.81961 0.93333 1" />
+      </material>
+    </visual>
+    <collision>
+      <origin
+        xyz="0 0 0"
+        rpy="1.5707963267949 0 0" />
+      <geometry>
+        <mesh filename="package://explorer_bot/models/world/meshes/wheel.stl" scale="0.8 0.8 0.8"/>
+      </geometry>
+    </collision>
+  </link>
+<link name="rear_left_wheel">
+    <inertial>
+      <origin
+        xyz="-4.1867E-18 0.0068085 -1.65658661799998E-18"
+        rpy="0 0 0" />
+      <mass
+        value="2.6578" />
+      <inertia
+        ixx="0.00856502765719703"
+        ixy="1.5074118157338E-19"
+        ixz="-4.78150098725052E-19"
+        iyy="0.013670640432096"
+        iyz="-2.68136447099727E-19"
+        izz="0.00856502765719703" />
+    </inertial>
+    <visual>
+      <origin
+        xyz="0 0 0"
+        rpy="1.5707963267949 0 0" />
+      <geometry>
+        <mesh filename="package://explorer_bot/models/world/meshes/wheel.stl" scale="0.8 0.8 0.8"/>
+      </geometry>
+      <material
+        name="">
+        <color
+          rgba="0.79216 0.81961 0.93333 1" />
+      </material>
+    </visual>
+    <collision>
+      <origin
+        xyz="0 0 0"
+        rpy="1.5707963267949 0 0" />
+      <geometry>
+        <mesh filename="package://explorer_bot/models/world/meshes/wheel.stl" scale="0.8 0.8 0.8"/>
+      </geometry>
+    </collision>
+  </link>
+<link name="rear_right_wheel">
+    <inertial>
+      <origin
+        xyz="-4.1867E-18 0.0068085 -1.65658661799998E-18"
+        rpy="0 0 0" />
+      <mass
+        value="2.6578" />
+      <inertia
+        ixx="0.00856502765719703"
+        ixy="1.5074118157338E-19"
+        ixz="-4.78150098725052E-19"
+        iyy="0.013670640432096"
+        iyz="-2.68136447099727E-19"
+        izz="0.00856502765719703" />
+    </inertial>
+    <visual>
+      <origin
+        xyz="0 0 0"
+        rpy="1.5707963267949 0 0" />
+      <geometry>
+        <mesh filename="package://explorer_bot/models/world/meshes/wheel.stl" scale="0.8 0.8 0.8"/>
+      </geometry>
+      <material
+        name="">
+        <color
+          rgba="0.79216 0.81961 0.93333 1" />
+      </material>
+    </visual>
+    <collision>
+      <origin
+        xyz="0 0 0"
+        rpy="1.5707963267949 0 0" />
+      <geometry>
+        <mesh filename="package://explorer_bot/models/world/meshes/wheel.stl" scale="0.8 0.8 0.8"/>
+      </geometry>
+    </collision>
+  </link>
+<joint name="front_left_wheel_joint" type="continuous">
+    <axis xyz="0 1 0"/>
+    <parent link ="base_link"/>
+    <child link ="front_left_wheel"/>
+    <origin rpy ="0 0 0" xyz= "0.176 0.205 0"/>
+  </joint>
+<joint name="front_right_wheel_joint" type="continuous">
+    <axis xyz="0 1 0"/>
+    <parent link ="base_link"/>
+    <child link ="front_right_wheel"/>
+    <origin rpy ="0 0 0" xyz= "0.176 -0.205 0"/>
+  </joint>
+<joint name="rear_left_wheel_joint" type="continuous">
+    <axis xyz="0 1 0"/>
+    <parent link ="base_link"/>
+    <child link ="rear_left_wheel"/>
+    <origin rpy ="0 0 0" xyz= "-0.176 0.205 0"/>
+  </joint>
+<joint name="rear_right_wheel_joint" type="continuous">
+    <axis xyz="0 1 0"/>
+    <parent link ="base_link"/>
+    <child link ="rear_right_wheel"/>
+    <origin rpy ="0 0 0" xyz= "-0.176 -0.205 0"/>
 </joint>
 <!--Front arm-->
@@ -468,4 +496,9 @@
   </gazebo>
 <!--######################################################################-->
+<gazebo>
+  <plugin name="joint_state_publisher" filename="libgazebo_ros_joint_state_publisher.so">
+    <jointName>arm_joint</jointName>
+  </plugin>
+</gazebo>
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
Commit message: final Dolly bot is ready to roll with teleop_keyboard

File: urdf/dolly.urdf.xacro (robot description, xacro)
@@ -76,5 +76,5 @@
   </inertial>
 </link>
-<joint name="arm_joint" type="continuous">
+<joint name="arm_joint" type="revolute">
   <parent link="base_link"/>
   <child link="arm_link"/>
@@ -86,16 +86,13 @@
 <link name="hand">
   <inertial>
-    <origin
-      xyz="7.7128E-09 -0.063005 -3.01969999961422E-08"
-      rpy="0 0 0" />
     <mass
       value="1.6004" />
     <inertia
-      ixx="0.00552196561445819"
-      ixy="7.9550614501301E-10"
-      ixz="-1.34378458924839E-09"
-      iyy="0.00352397447953875"
-      iyz="-1.10071809773382E-08"
-      izz="0.00553739792746489" />
+      ixx="0.0038550675"
+      ixy="0"
+      ixz="0"
+      iyy="0.0038550675"
+      iyz="0"
+      izz="0.0038550675" />
   </inertial>
   <visual>
@@ -121,8 +118,10 @@
   </collision>
 </link>
-<joint name="hand_joint" type="fixed">
-  <axis xyz="0 0 1"/>
+<joint name="hand_joint" type="revolute">
+  <axis xyz="0 1 0"/>
   <parent link="base_link"/>
   <child link="hand"/>
+  <dynamics damping="3.0" friction="0.3"/>
+  <limit effort="30.0" lower="-1.57079632679" upper="1.57079632679" velocity="5.0"/>
   <origin rpy="0 1.578 3.14" xyz="0.05 0.27 0.2"/>
 </joint>
@@ -498,5 +497,5 @@
 <gazebo>
   <plugin name="joint_state_publisher" filename="libgazebo_ros_joint_state_publisher.so">
-    <jointName>arm_joint</jointName>
+    <jointName>arm_joint,hand_joint</jointName>
   </plugin>
 </gazebo>
@@ -595,5 +594,5 @@
 <transmission name="arm_base_trans" type="SimpleTransmission">
   <type>transmission_interface/SimpleTransmission</type>
-  <actuator name="arm_base_motor">
+  <actuator name="arm_motor">
    <hardwareInterface>hardware_interface/PositionJointInterface</hardwareInterface>
    <mechanicalReduction>1</mechanicalReduction>
@@ -603,3 +602,13 @@
   </joint>
 </transmission>
+<transmission name="hand_base_trans" type="SimpleTransmission">
+  <type>transmission_interface/SimpleTransmission</type>
+  <actuator name="hand_motor">
+   <hardwareInterface>hardware_interface/PositionJointInterface</hardwareInterface>
+   <mechanicalReduction>1</mechanicalReduction>
+  </actuator>
+  <joint name="hand_joint">
+   <hardwareInterface>hardware_interface/PositionJointInterface</hardwareInterface>
+  </joint>
+</transmission>
 </robot>
